File: src/DataFusionExe/PressureReadings/PCB/WiiBoard/WiiBoard.kicad_pcb (KiCad board)
At the start: 2 copper layers, 7 parts, among them J1 Conn_01x04, J2 Conn_01x04, J3 Conn_01x04, J4 Conn_01x04, J5 Conn_01x20, J6 Conn_01x20

Commit message: PCB Corrections
Parts:
- added H1: MountingHole, MountingHole:MountingHole_3.2mm_M3, F.Cu at (132.1, 101.6)
- added H2: MountingHole, MountingHole:MountingHole_3.2mm_M3, F.Cu at (86.4, 43.2)
- added H3: MountingHole, MountingHole:MountingHole_3.2mm_M3, F.Cu at (86.4, 101.6)
- added MH 1: MountingHole, MountingHole:MountingHole_3.2mm_M3, F.Cu at (132.1, 43.2)
- C1: footprint Capacitor_THT:CP_Radial_D13.0mm_P5.00mm -> Capacitor_THT:CP_Radial_D8.0mm_P5.00mm
- moved J2 110.2 mm to (124.5, 62.0)
- moved J4 95.8 mm to (124.5, 48.9)
- moved C1 85.4 mm to (101.7, 86.4)
- moved J5 68.7 mm to (113.5, 49.7)
- moved J6 66.2 mm to (93.5, 49.7)
- moved J1 62.4 mm to (124.5, 90.2)
- moved J3 56.4 mm to (124.5, 76.2)
Routing:
- net Net-(J1-Pin_3): track 0.00 -> 93.3 mm, vias 0 -> 2
- net Net-(J2-Pin_2): track 0.00 -> 71.2 mm
- net Net-(J1-Pin_2): track 0.00 -> 66.6 mm, vias 0 -> 2
- net VDD: track 0.00 -> 64.5 mm, vias 0 -> 6
- net Net-(J4-Pin_2): track 0.00 -> 61.5 mm
- net +3.3V: track 0.00 -> 15.6 mm
- net Net-(J3-Pin_2): track 0.00 -> 12.5 mm
- added copper zone on B.Cu, net GND
Other:
- board outline added: 55.9 x 68.6 mm
